File: Hardware/Basic/Top/LowKey-BASIC-TOP.brd (EAGLE design)
At the start: 0 parts

Commit message: Added basic top board elements
Parts:
- added C10, C11: 300p, LinnesLab-Passives:C0603
- added C12: 10u, LinnesLab-Passives:C0805
- added C13, C15, C17, C18, C19: 2.2uF, LinnesLab-Passives:C0402
- added C14: 100n, LinnesLab-Passives:C0603
- added C16: 10uF, LinnesLab-Passives:C0603
- added C2, C5, C6, C7: 1u, LinnesLab-Passives:C0603
- added C20, C21: 4.7u, LinnesLab-Passives:C0603
- added C8, C9: (no value), LinnesLab-Passives:C0603
- added CHRG2: MCP73831, LinnesLab-Power:SOT23-5
- added CORTEX1: CORTEX_DEBUG_PTH, LinnesLab-Connectors:2X5-PTH-1.27MM
- added D1, D4, D5: (no value), LinnesLab-DiscreteSemi:USC
- added J2: (no value), LinnesLab-Connectors:1X02
- added L2: 10u, LinnesLab-Passives:L0603
- added LDO2: MIC5504, LinnesLab-Power:SOT23-5
- added LED3: RED, LinnesLab-LED:LED-0603
- added LED4: BLUE, LinnesLab-LED:LED-0603
- added R11: (no value), LinnesLab-Passives:R0603
- added R12, R13, R14, R15: 100k, LinnesLab-Passives:R0603
- added R3, R4: 1k, LinnesLab-Passives:R0603
- added R5, R6, R8, R9: 10k, LinnesLab-Passives:R0603
- added R7: 390k, LinnesLab-Passives:R0603
- added SD2: (no value), LinnesLab-Connectors:MICROSD
- added SW1, SW2, SW5: SWITCH.MOM, LinnesLab-Switches:TACTILE_SWITCH_SMD_6.2MM_TALL
- added SW3, SW4: (no value), LinnesLab-Switches:BUTTON-GULLWING
- added U2: NRF52832_MODULE_MDBT42, LinnesLab-Microcontrollers:BLE_MODULE_RAYTAC_MDBT42
- added U3: (no value), LinnesLab-Displays:UG-2864HSWEG01_0.96IN_NO-WRAPAROUND
- added U4: PCF8523, LinnesLab-Clocks:SO8
- added USB2: USB.MICRO-BIGGERPADS, LinnesLab-Connectors:USB-MICRO-01.BIGGERPADS
- added XTAL2: 32.768kHz, LinnesLab-Clocks:2-SMD.NOLEAD.2.0MMTO1.2MM
- added XTAL3: 32.7680kHz, LinnesLab-Clocks:2-SMD.NOLEAD.2.0MMTO1.2MM
Connections:
- new net 3.3V: C12.2, C17.2, C19.2, C2.1, C6.1, CORTEX1.1, D1.-, LDO2.5, R15.2, R5.2, R8.2, R9.2, SD2.4, U2.11, U3.6, U3.9, U4.8
- new net BATT: R13.1, R14.2
- new net CD1: SD2.CD1
- new net CD2: SD2.CD2
- new net CHRG.STAT: CHRG2.1, R12.1
- new net CS.OLED: U3.13
- new net DC.OLED: U3.15
- new net DFU: SW3.3, U2.34
- new net DTR: C14.1
- new net FRST: U2.38
- new net GND: C10.2, C11.2, C12.1, C16.1, C17.1, C18.1, C19.1, C2.2, C20.2, C21.1, C5.1, C6.2, C7.2, C8.1, C9.2, CHRG2.2, CORTEX1.3, CORTEX1.5, CORTEX1.7, CORTEX1.9, J2.1, LDO2.2, LED3.C, LED4.C, R11.1, R14.1, R15.1, R6.1, R7.2, SD2.6, SD2.MT1, SD2.MT2, SW1.B1, SW1.B2, SW2.B1, SW2.B2, SW3.1, SW4.3, SW5.B1, SW5.B2, U2.1, U2.12, U2.24, U2.39, U3.1, U3.10, U3.12, U3.29, U3.30, U3.8, U4.4, USB2.5
- new net LED1: R3.2, U2.31
- new net LED2: R4.2, U2.33
- new net MISO: SD2.7, U2.28
- new net MOSI: SD2.3, U2.27, U3.19
- new net N$1: R6.2, U3.11
- new net N$10: LED4.A, R4.1
- new net N$11: L2.1, U2.10
- new net N$12: C7.1, L2.2, U2.9
- new net N$13: C16.2, U3.28
- new net N$14: CORTEX1.8
- new net N$15: C18.2, U3.27
- new net N$17: CHRG2.5, R11.2
- new net N$19: U4.2, XTAL3.P$1
- new net N$2: R7.1, U3.26
- new net N$20: U4.1, XTAL3.P$2
- new net N$3: C13.2, U3.2
- new net N$4: C8.2, U2.13, XTAL2.P$1
- new net N$5: C13.1, U3.3
- new net N$6: C9.1, U2.14, XTAL2.P$2
- new net N$7: C15.2, U3.4
- new net N$8: C15.1, U3.5
- new net N$9: LED3.A, R3.1
- new net P0.09/NFC1: C11.1, U2.22
- new net P0.10/NFC2: C10.1, U2.23
- new net RESET: C14.2, CORTEX1.10, D1.+, R5.1, SW4.1, U2.35
- new net RESET.OLED: U3.14
- new net RXD: U2.21
- new net SCK: SD2.5, U2.26, U3.18
- new net SCL: R8.1, U2.3, U4.6
- new net SD.CS: SD2.2
- new net SDA: R9.1, U2.2, U4.5
- new net SW1: SW1.A1, SW1.A2, SW2.A1, SW2.A2, SW5.A1, SW5.A2
- new net SWCLK: CORTEX1.4, U2.36
- new net SWDIO: CORTEX1.2, U2.37
- new net SWO: CORTEX1.6, U2.32
- new net TXD: U2.19
- new net USB+: USB2.3
- new net USB-: USB2.2
- new net VBATT: U4.3
- new net VIN: C21.2, C5.2, CHRG2.4, D4.-, D5.-, LDO2.1, LDO2.3, R12.2
- new net VLIPO: C20.1, CHRG2.3, D4.+, J2.2, R13.2
- new net V_USB: D5.+, USB2.1
Other:
- board outline added: 38 x 38 mm

Commit message: Top connections
Parts:
- added C22: 100n, LinnesLab-Passives:C0603
- added C23, C24: 47p, LinnesLab-Passives:C0603
- added J1: (no value), LinnesLab-Connectors:1X07
- added JP2: (no value), LinnesLab-Switches:SMT-JUMPER_2_NO_SILK
- added LED5: RED, LinnesLab-LED:LED-0603
- added LED6: YELLOW, LinnesLab-LED:LED-0603
- added R1, R2: 0, LinnesLab-Passives:R0603
- added R17, R18: 27, LinnesLab-Passives:R0603
- added R19, R20: 1k, LinnesLab-Passives:R0603
- added U5: FT231XS, LinnesLab-DigitalIC:SSOP20_L
- moved R9 63.1 mm to (0.46, -26.7), turned to 0 degrees
- moved R8 59.3 mm to (0.46, -24.0), turned to 0 degrees
- moved U4 50.3 mm to (13.2, -18.3)
- moved XTAL3 50.3 mm to (8.61, -16.8)
- moved C2 48.3 mm to (15.0, -14.7)
- moved C16 5.39 mm to (24.4, 30.9)
- moved C18 5.35 mm to (12.9, 30.1)
- moved C12 5.09 mm to (9.58, 30.0)
- moved U3 4.40 mm to (17.0, 19.9)
- moved C13 3.50 mm to (7.54, 23.9)
- moved C15 3.40 mm to (8.84, 23.9)
- moved C19 3.27 mm to (10.2, 23.9)
- moved C17 3.12 mm to (11.5, 24.0)
- moved U2 0.78 mm to (31.5, 29.3)
Connections:
- net VBATT renamed VBAT
- removed net BATT: R13.1, R14.2
- removed net CD1: SD2.CD1
- removed net CHRG.STAT: CHRG2.1, R12.1
- removed net CS.OLED: U3.13
- removed net DC.OLED: U3.15
- removed net RESET.OLED: U3.14
- removed net RXD: U2.21
- removed net SD.CS: SD2.2
- removed net SW1: SW1.A1, SW1.A2, SW2.A1, SW2.A2, SW5.A1, SW5.A2
- removed net TXD: U2.19
- new net !CTS: JP2.2, U5.9
- new net A4/BATT: R13.1, R14.2, U2.5
- new net A6/TIA: U2.7
- new net A7/PPG: U2.8
- new net D11/SW1: SW1.A1, SW1.A2, U2.25
- new net D15/SW2: SW2.A1, SW2.A2, U2.29
- new net D16/CS.OLED: U2.30, U3.13
- new net D27/CHRG.STATUS: CHRG2.1, R12.1, U2.4
- new net D29/LED.CTRL: U2.6
- new net D3/RESET.OLED: U2.16, U3.14
- new net D4/DC.OLED: U2.17, U3.15
- new net D5/CD1: SD2.CD1, U2.18
- new net D7/SD.CS: SD2.2, U2.20
- new net FT3V3: U5.13
- new net N$29: R17.2, U5.12
- new net N$30: R18.2, U5.11
- new net N$31: LED5.C, R19.2
- new net N$32: LED6.C, R20.2
- new net RXD.FT: R2.1, U5.4
- new net RXD.NRF: R1.2, U2.21
- new net RXLED: R19.1, U5.17
- new net SW3: SW5.A1, SW5.A2
- new net TXD.FT: R1.1, U5.20
- new net TXD.NRF: R2.2, U2.19
- new net TXLED: R20.1, U5.10
- net 3.3V: now also C22.2, LED5.A, LED6.A, U5.14, U5.3
- net DTR: now also U5.1
- net GND: now also C22.1, C23.2, C24.1, JP2.1, U5.16, U5.6
- net SCL: now also R9.1; no longer R8.1
- net SDA: now also R8.1; no longer R9.1
- net USB+: now also C23.1, R18.1
- net USB-: now also C24.2, R17.1
- net V_USB: now also U5.15

Commit message: Take 4 Routing Top Board 17 min
Parts:
- removed C22: 100n, LinnesLab-Passives:C0603
- removed C23, C24: 47p, LinnesLab-Passives:C0603
- removed CHRG2: MCP73831, LinnesLab-Power:SOT23-5
- removed D4, D5: (no value), LinnesLab-DiscreteSemi:USC
- removed JP2: (no value), LinnesLab-Switches:SMT-JUMPER_2_NO_SILK
- removed L2: 10u, LinnesLab-Passives:L0603
- removed LDO2: MIC5504, LinnesLab-Power:SOT23-5
- removed LED5: RED, LinnesLab-LED:LED-0603
- removed LED6: YELLOW, LinnesLab-LED:LED-0603
- removed R19, R20: 1k, LinnesLab-Passives:R0603
- removed U5: FT231XS, LinnesLab-DigitalIC:SSOP20_L
- removed XTAL3: 32.7680kHz, LinnesLab-Clocks:2-SMD.NOLEAD.2.0MMTO1.2MM
- added C1: 1u, LinnesLab-Passives:C0603
- added C3: 47p, LinnesLab-Passives:C0603
- added C4: 10u, LinnesLab-Passives:C0805
- added CHRG1: MCP73831, LinnesLab-Power:SOT23-5
- added D2, D3: (no value), LinnesLab-DiscreteSemi:USC
- added JP1: (no value), LinnesLab-Switches:SMT-JUMPER_2_NO_SILK
- added L1: 10u, LinnesLab-Passives:L0603
- added LDO1: MIC5504, LinnesLab-Power:SOT23-5
- added LED1, LED2: RED, LinnesLab-LED:LED-0603
- added R10: 1k, LinnesLab-Passives:R0603
- added R16: 10k, LinnesLab-Passives:R0603
- added U1: NRF52832_MODULE_MDBT42, LinnesLab-Microcontrollers:BLE_MODULE_RAYTAC_MDBT42
- added XTAL1: 32.768kHz, LinnesLab-Clocks:2-SMD.NOLEAD.2.0MMTO1.2MM
- C12: value 10u -> 1u; device LinnesLab-Passives:C0805 -> LinnesLab-Passives:C0603
- C13: value 2.2uF -> 4.7u; device LinnesLab-Passives:C0402 -> LinnesLab-Passives:C0603
- C15: value 2.2uF -> 10uF; device LinnesLab-Passives:C0402 -> LinnesLab-Passives:C0603
- C16: value 10uF -> 2.2uF; device LinnesLab-Passives:C0603 -> LinnesLab-Passives:C0402
- C2: value 1u -> 47p
- C20: value 4.7u -> 2.2uF; device LinnesLab-Passives:C0603 -> LinnesLab-Passives:C0402
- C21: value 4.7u -> 1u
- C5: value 1u -> (none)
- C6: value 1u -> 100n
- C7: value 1u -> 4.7u
- C8: value (none) -> 1u
- J1: device LinnesLab-Connectors:1X07 -> LinnesLab-Connectors:1X07_1.27MM
- LED3: value RED -> YELLOW
- R1, R2: value 0 -> 10k
- R11: value (none) -> 1k
- R14, R15: value 100k -> 0
- R17: value 27 -> 10k
- R18: value 27 -> 390k
- R3, R4: value 1k -> 27
- R5: value 10k -> 100k
- R6: value 10k -> (none)
- R7: value 390k -> 100k
- R8, R9: value 10k -> 1k
- SW1, SW2: value SWITCH.MOM -> (none); device LinnesLab-Switches:TACTILE_SWITCH_SMD_6.2MM_TALL -> LinnesLab-Switches:BUTTON-GULLWING
- SW3, SW4: value (none) -> SWITCH.MOM; device LinnesLab-Switches:BUTTON-GULLWING -> LinnesLab-Switches:TACTILE_SWITCH_SMD_6.2MM_TALL
- U2: value NRF52832_MODULE_MDBT42 -> FT231XS; device LinnesLab-Microcontrollers:BLE_MODULE_RAYTAC_MDBT42 -> LinnesLab-DigitalIC:SSOP20_L
- U3: value (none) -> PCF8523; device LinnesLab-Displays:UG-2864HSWEG01_0.96IN_NO-WRAPAROUND -> LinnesLab-Clocks:SO8
- U4: value PCF8523 -> (none); device LinnesLab-Clocks:SO8 -> LinnesLab-Displays:UG-2864HSWEG01_0.96IN_NO-WRAPAROUND
- XTAL2: value 32.768kHz -> 32.7680kHz
- moved R8 86.1 mm to (35.7, 54.5)
- moved SW3 72.9 mm to (-16.5, -0.03)
- moved C2 70.8 mm to (38.2, 52.2), turned to 270 degrees
- moved R9 65.8 mm to (40.1, 25.8), turned to 180 degrees
- moved R14 56.0 mm to (28.2, 60.0), turned to 0 degrees
- moved C6 55.2 mm to (24.0, 55.7)
- moved R17 55.0 mm to (14.3, 27.4), turned to 90 degrees
- moved R15 54.4 mm to (34.2, 60.3), turned to 0 degrees
- moved R18 52.4 mm to (17.1, 27.2), turned to 90 degrees
- moved U3 49.6 mm to (41.5, -23.2)
- moved SW1 48.0 mm to (49.4, 31.2)
- moved C14 45.1 mm to (66.2, -22.9)
- moved R2 44.5 mm to (11.8, 27.7), turned to 90 degrees
- moved C13 41.9 mm to (31.3, -10.7)
- moved R1 41.5 mm to (8.87, 28.0), turned to 90 degrees
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- renumbered CORTEX1 to DEBUG1, SD2 to SD1, USB2 to USB1
Connections:
- net !CTS: now also JP1.2, U2.9; no longer JP2.2, U5.9
- net 3.3V: now also C12.1, C20.2, C21.1, C4.2, C6.2, D3.-, J1.4, LDO1.5, LED1.A, LED3.A, R1.2, R16.2, R2.2, R7.2, U1.11, U2.14, U2.3, U3.8, U4.6, U4.9; no longer C12.2, C17.2, C2.1, C22.2, C6.1, D1.-, LDO2.5, LED5.A, LED6.A, R15.2, R5.2, R8.2, R9.2, U2.11, U3.6, U3.9, U4.8, U5.14, U5.3
- net A4/BATT: now also R12.1, R13.2, U1.5; no longer R13.1, R14.2, U2.5
- net A6/TIA: now also J1.6, U1.7; no longer U2.7
- net A7/PPG: now also J1.7, U1.8; no longer U2.8
- net D11/SW1: now also SW3.A1, SW3.A2, U1.25; no longer SW1.A1, SW1.A2, U2.25
- net D15/SW2: now also SW4.A1, SW4.A2, U1.29; no longer SW2.A1, SW2.A2, U2.29
- net D16/CS.OLED: now also U1.30, U4.13; no longer U2.30, U3.13
- net D27/CHRG.STATUS: now also CHRG1.1, R5.1, U1.4; no longer CHRG2.1, R12.1, U2.4
- net D29/LED.CTRL: now also J1.5, U1.6; no longer U2.6
- net D3/RESET.OLED: now also U1.16, U4.14; no longer U2.16, U3.14
- net D4/DC.OLED: now also U1.17, U4.15; no longer U2.17, U3.15
- net D5/CD1: now also U1.18; no longer U2.18
- net D7/SD.CS: now also U1.20; no longer U2.20
- net DFU: now also SW1.3, U1.34; no longer SW3.3, U2.34
- net DTR: now also U2.1; no longer U5.1
- net FRST: now also U1.38; no longer U2.38
- net FT3V3: now also U2.13; no longer U5.13
- net GND: now also C1.2, C12.2, C13.2, C15.1, C2.1, C20.1, C21.2, C3.2, C4.1, C6.1, C7.1, CHRG1.2, J1.3, JP1.1, LDO1.2, LED2.C, R13.1, R17.1, R18.2, R7.1, SW1.1, SW2.3, SW3.B1, SW3.B2, SW4.B1, SW4.B2, U1.1, U1.12, U1.24, U1.39, U2.16, U2.6, U3.4, U4.1, U4.10, U4.12, U4.29, U4.30, U4.8; no longer C12.1, C16.1, C18.1, C2.2, C20.2, C21.1, C22.1, C23.2, C24.1, C6.2, C7.2, CHRG2.2, JP2.1, LDO2.2, LED3.C, R11.1, R14.1, R15.1, R7.2, SW1.B1, SW1.B2, SW2.B1, SW2.B2, SW3.1, SW4.3, U2.1, U2.12, U2.24, U2.39, U3.1, U3.10, U3.12, U3.29, U3.30, U3.8, U4.4, U5.16, U5.6
- net LED1: now also R9.2, U1.31; no longer R3.2, U2.31
- net LED2: now also R11.2, U1.33; no longer R4.2, U2.33
- net MISO: now also U1.28; no longer U2.28
- net MOSI: now also U1.27, U4.19; no longer U2.27, U3.19
- net N$1: now also R17.2, U4.11; no longer R6.2, U3.11
- net N$10: now also R11.1; no longer R4.1
- net N$11: now also L1.1, U1.10; no longer L2.1, U2.10
- net N$12: now also C1.1, L1.2, U1.9; no longer C7.1, L2.2, U2.9
- net N$13: now also C15.2, U4.28; no longer C16.2, U3.28
- net N$15: now also C17.2, U4.27; no longer C18.2, U3.27
- net N$17: now also CHRG1.5, R6.2; no longer CHRG2.5, R11.2
- net N$2: now also R18.1, U4.26; no longer R7.1, U3.26
- net N$25: now also U3.2, XTAL2.P$1; no longer U4.2, XTAL3.P$1
- net N$26: now also U3.1, XTAL2.P$2; no longer U4.1, XTAL3.P$2
- net N$29: now also R3.2, U2.12; no longer R17.2, U5.12
- net N$3: now also C18.2, U4.2; no longer C13.2, U3.2
- net N$30: now also R4.2, U2.11; no longer R18.2, U5.11
- net N$31: now also LED1.C, R8.2; no longer LED5.C, R19.2
- net N$32: now also LED3.C, R10.2; no longer LED6.C, R20.2
- net N$4: now also C5.2, U1.13, XTAL1.P$1; no longer C8.2, U2.13, XTAL2.P$1
- net N$5: now also C18.1, U4.3; no longer C13.1, U3.3
- net N$6: now also U1.14, XTAL1.P$2; no longer U2.14, XTAL2.P$2
- net N$7: now also C16.2, U4.4; no longer C15.2, U3.4
- net N$8: now also C16.1, U4.5; no longer C15.1, U3.5
- net N$9: now also LED2.A, R9.1; no longer LED3.A, R3.1
- net P0.09/NFC1: now also C10.1, U1.22; no longer C11.1, U2.22
- net P0.10/NFC2: now also C11.1, U1.23; no longer C10.1, U2.23
- net RESET: now also D3.+, R16.1, SW2.1, U1.35; no longer D1.+, R5.1, SW4.1, U2.35
- net RXD.FT: now also R14.1, U2.4; no longer R2.1, U5.4
- net RXD.NRF: now also R15.2, U1.21; no longer R1.2, U2.21
- net RXLED: now also R8.1, U2.17; no longer R19.1, U5.17
- net SCK: now also U1.26, U4.18; no longer U2.26, U3.18
- net SCL: now also J1.2, R2.1, U1.3, U3.6; no longer R9.1, U2.3, U4.6
- net SDA: now also J1.1, R1.1, U1.2, U3.5; no longer R8.1, U2.2, U4.5
- net SWCLK: now also U1.36; no longer U2.36
- net SWDIO: now also U1.37; no longer U2.37
- net SWO: now also U1.32; no longer U2.32
- net TXD.FT: now also R15.1, U2.20; no longer R1.1, U5.20
- net TXD.NRF: now also R14.2, U1.19; no longer R2.2, U2.19
- net TXLED: now also R10.1, U2.10; no longer R20.1, U5.10
- net USB+: now also C3.1, R4.1; no longer C23.1, R18.1
- net USB-: now also C2.2, R3.1; no longer C24.2, R17.1
- net VBAT: now also U3.3; no longer U4.3
- net VIN: now also C7.2, C8.2, CHRG1.4, D1.-, D2.-, LDO1.1, LDO1.3, R5.2; no longer C21.2, C5.2, CHRG2.4, D4.-, D5.-, LDO2.1, LDO2.3, R12.2
- net VLIPO: now also C13.1, CHRG1.3, D1.+, R12.2; no longer C20.1, CHRG2.3, D4.+, R13.2
- net V_USB: now also D2.+, U2.15; no longer D5.+, U5.15
Routing:
- net TXLED: track 0.00 -> 13.6 mm, vias 0 -> 2
- net GND: track 0.00 -> 9.13 mm, vias 0 -> 2
- net RXD.FT: track 0.00 -> 8.81 mm
- net N$12: track 0.00 -> 4.79 mm
- net TXD.FT: track 0.00 -> 4.02 mm
- net N$30: track 0.00 -> 2.82 mm
- net 3.3V: track 0.00 -> 2.80 mm
- net N$11: track 0.00 -> 2.50 mm
- net N$31: track 0.00 -> 2.10 mm
- net N$32: track 0.00 -> 1.98 mm
- net N$29: track 0.00 -> 1.92 mm
- net RXLED: track 0.00 -> 1.71 mm
- net USB+: track 0.00 -> 1.66 mm
- net USB-: track 0.00 -> 1.49 mm
- added copper zone on layer 1, net 3.3V
- added copper zone on layer 16, net GND

Commit message: Take 4 Complete
Parts:
- removed C10, C11: 300p, LinnesLab-Passives:C0603
- removed R7: 100k, LinnesLab-Passives:R0603
- moved JP1 99.8 mm to (-5.81, -24.4), turned to 90 degrees
- moved C2 79.8 mm to (5.96, -20.8)
- moved C3 79.8 mm to (6.11, -24.3)
- moved LED1 79.8 mm to (7.23, -18.4)
- moved LED3 79.8 mm to (7.15, -15.7)
- moved R10 79.8 mm to (3.45, -15.6)
- moved R14 79.8 mm to (-4.04, -12.9)
- moved R15 79.8 mm to (1.93, -12.6)
- moved R3 79.8 mm to (3.62, -21.6)
- moved R8 79.8 mm to (3.41, -18.4)
- moved U2 79.8 mm to (-1.82, -19.4)
- moved R4 79.8 mm to (3.64, -23.6)
- moved C6 79.5 mm to (-5.74, -18.0), turned to 90 degrees
- moved SW3 48.2 mm to (31.5, 4.25)
- moved SW5 32.4 mm to (-10.5, -4.06)
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Connections:
- net 3.3V: no longer R7.2
- net GND: no longer C10.2, C11.2, R7.1, SW3.B2, SW4.B2
- net P0.09/NFC1: no longer C10.1
- net P0.10/NFC2: no longer C11.1
Routing:
- net GND: track 9.13 -> 34.2 mm, vias 2 -> 14
- net VLIPO: track 0.00 -> 13.3 mm
- net TXLED: track 13.6 -> 1.51 mm, vias 2 -> 1
- net VIN: track 0.00 -> 8.46 mm
- net N$2: track 0.00 -> 6.26 mm
- net N$13: track 0.00 -> 6.21 mm
- net SWDIO: track 0.00 -> 6.15 mm
- net N$8: track 0.00 -> 6.04 mm
- net N$15: track 0.00 -> 4.52 mm
- net N$3: track 0.00 -> 4.11 mm
- net N$5: track 0.00 -> 3.86 mm
- net N$7: track 0.00 -> 3.82 mm
- net N$1: track 0.00 -> 3.13 mm
- net V_USB: track 0.00 -> 2.52 mm
- net 3.3V: track 2.80 -> 5.11 mm, vias 0 -> 1
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
Commit message: Take 06
Parts:
- removed C12, C21, C8: 1u, LinnesLab-Passives:C0603
- removed C13, C7: 4.7u, LinnesLab-Passives:C0603
- removed CHRG1: MCP73831, LinnesLab-Power:SOT23-5
- removed LDO1: MIC5504, LinnesLab-Power:SOT23-5
- removed R5: 100k, LinnesLab-Passives:R0603
- removed R6: (no value), LinnesLab-Passives:R0603
- removed SD1: (no value), LinnesLab-Connectors:MICROSD
- removed U3: PCF8523, LinnesLab-Clocks:SO8
- removed XTAL2: 32.7680kHz, LinnesLab-Clocks:2-SMD.NOLEAD.2.0MMTO1.2MM
- moved R13 53.9 mm to (1.93, 23.1), turned to 90 degrees
- moved R12 49.6 mm to (3.80, 23.1), turned to 270 degrees
- moved SW2 45.6 mm to (34.3, 16.5), turned to 90 degrees
- moved C14 45.4 mm to (34.2, 9.29), turned to 0 degrees
- moved D3 45.1 mm to (34.2, 11.3), turned to 180 degrees
- moved R16 44.8 mm to (34.4, 13.2), flipped to the bottom, turned to 180 degrees
- moved C5 36.2 mm to (16.5, 22.5), turned to 270 degrees
- moved XTAL1 29.9 mm to (19.5, 22.2), turned to 90 degrees
- moved C2 29.6 mm to (16.0, 7.06)
- moved R3 29.6 mm to (13.3, 6.34)
- moved C9 29.4 mm to (17.8, 22.6), turned to 90 degrees
- moved C6 29.3 mm to (1.58, 10.4)
- moved C3 29.3 mm to (14.8, 3.60), turned to 90 degrees
- moved JP1 28.9 mm to (3.40, 2.97)
- moved R14 28.9 mm to (5.17, 14.5)
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Connections:
- removed net CD2: SD1.CD2
- removed net N$17: CHRG1.5, R6.2
- removed net N$25: U3.2, XTAL2.P$1
- removed net N$26: U3.1, XTAL2.P$2
- removed net VBAT: U3.3
- net 3.3V: no longer C12.1, C21.1, LDO1.5, SD1.4, U3.8
- net D27/CHRG.STATUS: no longer CHRG1.1, R5.1
- net D5/CD1: no longer SD1.CD1
- net D7/SD.CS: no longer SD1.2
- net GND: no longer C12.2, C13.2, C21.2, C7.1, C8.1, CHRG1.2, LDO1.2, R6.1, SD1.6, SD1.MT1, SD1.MT2, U3.4
- net MISO: no longer SD1.7
- net MOSI: no longer SD1.3
- net SCK: no longer SD1.5
- net SCL: no longer U3.6
- net SDA: no longer U3.5
- net VIN: no longer C7.2, C8.2, CHRG1.4, LDO1.1, LDO1.3, R5.2
- net VLIPO: no longer C13.1, CHRG1.3
Routing:
- net RESET: track 0.00 -> 36.4 mm, vias 0 -> 3
- net USB-: track 1.49 -> 22.9 mm, vias 0 -> 1
- net GND: track 34.2 -> 55.4 mm, vias 14 -> 20
- net USB+: track 1.66 -> 19.2 mm, vias 0 -> 1
- net SWO: track 0.00 -> 11.7 mm, vias 0 -> 1
- net VLIPO: track 13.3 -> 23.4 mm
- net SWCLK: track 0.00 -> 9.27 mm
- net RXD.FT: track 8.81 -> 0.00 mm
- net N$4: track 0.00 -> 8.44 mm
- net N$6: track 0.00 -> 7.65 mm
- net LED2: track 0.00 -> 7.41 mm
- net LED1: track 0.00 -> 4.14 mm
- net N$15: track 4.52 -> 1.01 mm
- net N$29: track 1.92 -> 5.22 mm
- net 3.3V: track 5.11 -> 1.85 mm, vias 1 -> 0
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
Commit message: Take 7
Parts:
- C17: device LinnesLab-Passives:C0402 -> LinnesLab-Passives:C0603
- moved SW3 10.3 mm to (21.9, 4.47)
- moved SW4 10.2 mm to (32.2, 4.49)
- moved C17 8.79 mm to (28.7, 13.7), turned to 180 degrees
- moved R2 7.03 mm to (3.41, 32.5), turned to 270 degrees
- moved C4 5.21 mm to (17.8, 33.2), turned to 0 degrees
- moved R1 4.91 mm to (1.96, 32.6), turned to 270 degrees
- moved L1 3.55 mm to (17.4, 30.0), turned to 0 degrees
- moved R15 2.88 mm to (13.9, 13.9)
- moved C1 2.41 mm to (17.3, 31.6), turned to 180 degrees
- moved C6 0.80 mm to (1.54, 9.62), turned to 270 degrees
- moved JP1 0.68 mm to (2.91, 2.50)
- moved C5 0.65 mm to (16.5, 23.2)
- moved C9 0.61 mm to (18.0, 23.2)
- moved SW1 0.50 mm to (33.9, 35.6), turned to 180 degrees
- moved XTAL1 0.49 mm to (19.7, 22.7)
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Connections:
- removed net A4/BATT: R12.1, R13.2, U1.5
- removed net A6/TIA: J1.6, U1.7
- removed net A7/PPG: J1.7, U1.8
- removed net D29/LED.CTRL: J1.5, U1.6
- new net A4/PPG: J1.7, U1.5
- new net A5/TIA: J1.6, U1.6
- new net A7/BATT: R12.1, R13.2, U1.8
- new net D30/LED.CTRL: J1.5, U1.7
Routing:
- net D15/SW2: track 0.00 -> 29.3 mm, vias 0 -> 2
- net A7/BATT: track 0.00 -> 27.4 mm, vias 0 -> 2
- net D11/SW1: track 0.00 -> 24.6 mm
- net D16/CS.OLED: track 0.00 -> 19.3 mm, vias 0 -> 2
- net SDA: track 0.00 -> 18.4 mm, vias 0 -> 1
- net SCK: track 0.00 -> 18.4 mm, vias 0 -> 2
- net SCL: track 0.00 -> 17.9 mm, vias 0 -> 1
- net MOSI: track 0.00 -> 17.8 mm, vias 0 -> 2
- net D30/LED.CTRL: track 0.00 -> 13.5 mm, vias 0 -> 1
- net DFU: track 0.00 -> 13.3 mm, vias 0 -> 2
- net D4/DC.OLED: track 0.00 -> 12.9 mm, vias 0 -> 2
- net D3/RESET.OLED: track 0.00 -> 12.7 mm, vias 0 -> 2
- net A5/TIA: track 0.00 -> 12.3 mm, vias 0 -> 1
- net A4/PPG: track 0.00 -> 11.0 mm, vias 0 -> 1
- net N$11: track 2.40 -> 8.01 mm
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