File: Hardware/Basic/Top/LowKey-BASIC-TOP.sch (EAGLE design)
At the start: 52 parts, among them SW1 SWITCH.MOM, SW2 SWITCH.MOM, SW5 SWITCH.MOM, U2 NRF52832_MODULE_MDBT42, U4 PCF8523

Commit message: Top connections
Parts:
- added C22: 100n, LinnesLab-Passives:CAPACITOR0603
- added C23, C24: 47p, LinnesLab-Passives:CAPACITOR0603
- added J1: (no value), LinnesLab-Connectors:CONN_07
- added JP2: (no value), LinnesLab-Switches:JUMPER-SMT_2_NO_SILK
- added LED5: RED, LinnesLab-LED:LED0603
- added LED6: YELLOW, LinnesLab-LED:LED0603
- added R1, R2: 0, LinnesLab-Passives:RESISTOR0603
- added R17, R18: 27, LinnesLab-Passives:RESISTOR0603
- added R19, R20: 1k, LinnesLab-Passives:RESISTOR0603
- added U5: FT231XS, LinnesLab-DigitalIC:FT231XS
Connections:
- removed net BATT: R13.1, R14.2
- removed net CD1: SD2.CARD_DETECT
- removed net CHRG.STAT: CHRG2.STAT, R12.1
- removed net CS.OLED: U3./CS
- removed net DC.OLED: U3.DC/I2C_SA0
- removed net RESET.OLED: U3./RES
- removed net RXD: U2.P0.08
- removed net SD.CS: SD2.CS
- removed net SW1: SW1.1, SW1.2, SW2.1, SW2.2, SW5.1, SW5.2
- removed net TXD: U2.P0.06
- removed net VBATT: U4.VBAT
- new net !CTS: JP2.2, U5.!CTS
- new net A4/BATT: R13.1, R14.2, U2.P0.28/AIN4
- new net A6/TIA: U2.P0.30/AIN6
- new net A7/PPG: U2.P0.31/AIN7
- new net D11/SW1: SW1.1, SW1.2, U2.P0.11
- new net D15/SW2: SW2.1, SW2.2, U2.P0.15
- new net D16/CS.OLED: U2.P0.16, U3./CS
- new net D27/CHRG.STATUS: CHRG2.STAT, R12.1, U2.P0.27
- new net D29/LED.CTRL: U2.P0.29/AIN5
- new net D3/RESET.OLED: U2.P0.03/AIN1, U3./RES
- new net D4/DC.OLED: U2.P0.04/AIN2, U3.DC/I2C_SA0
- new net D5/CD1: SD2.CARD_DETECT, U2.P0.05/AIN3
- new net D7/SD.CS: SD2.CS, U2.P0.07
- new net FT3V3: U5.3V3OUT
- new net N$29: R17.2, U5.USBDM
- new net N$30: R18.2, U5.USBDP
- new net N$31: LED5.C, R19.2
- new net N$32: LED6.C, R20.2
- new net RXD.FT: R2.1, U5.RXD
- new net RXD.NRF: R1.2, U2.P0.08
- new net RXLED: R19.1, U5.CBUS1
- new net SW3: SW5.1, SW5.2
- new net TXD.FT: R1.1, U5.TXD
- new net TXD.NRF: R2.2, U2.P0.06
- new net TXLED: R20.1, U5.CBUS2
- net 3.3V: now also C22.2, LED5.A, LED6.A, U5.!RESET, U5.VCCIO
- net DTR: now also U5.!DTR
- net GND: now also C22.1, C23.2, C24.1, JP2.1, U5.GND@16, U5.GND@6
- net SCL: now also R9.1; no longer R8.1
- net SDA: now also R8.1; no longer R9.1
- net USB+: now also C23.1, R18.1
- net USB-: now also C24.2, R17.1
- net V_USB: now also U5.VCC
Other:
- note added: "Back-up battery if desired"
- note added: "FTDI Serial-to-USB COnverter"
- note added: "I don't remember if CTS needs to be grounded or left floating so here's a jumper to ground so it can be configued either way dynamically."
- note added: "TXD goes to RX on the other device RXD goes to TX on the other device"
- moved on the sheet: C2, R8, R9, U4, XTAL3

Commit message: Take 4 Routing Top Board 17 min
Parts:
- removed C22: 100n, LinnesLab-Passives:CAPACITOR0603
- removed C24: 47p, LinnesLab-Passives:CAPACITOR0603
- removed D4: (no value), LinnesLab-DiscreteSemi:SCHOTTKY-USC
- removed LED6: YELLOW, LinnesLab-LED:LED0603
- removed R19: 1k, LinnesLab-Passives:RESISTOR0603
- removed U5: FT231XS, LinnesLab-DigitalIC:FT231XS
- removed XTAL3: 32.7680kHz, LinnesLab-Clocks:CRYSTALECS-.327-12.5-12-C-TR
- added C1: 1u, LinnesLab-Passives:CAPACITOR0603
- added C4: 10u, LinnesLab-Passives:CAPACITOR0805
- added D3: (no value), LinnesLab-DiscreteSemi:SCHOTTKY-USC
- added LED2: RED, LinnesLab-LED:LED0603
- added R16: 10k, LinnesLab-Passives:RESISTOR0603
- added U1: NRF52832_MODULE_MDBT42, LinnesLab-Microcontrollers:NRF52832_MODULE_MDBT42
- added XTAL1: 32.768kHz, LinnesLab-Clocks:CRYSTALECS-.327-12.5-12-C-TR
- C12: value 10u -> 1u; device LinnesLab-Passives:CAPACITOR0805 -> LinnesLab-Passives:CAPACITOR0603
- C13: value 2.2uF -> 4.7u; device LinnesLab-Passives:CAPACITOR0402 -> LinnesLab-Passives:CAPACITOR0603
- C15: value 2.2uF -> 10uF; device LinnesLab-Passives:CAPACITOR0402 -> LinnesLab-Passives:CAPACITOR0603
- C16: value 10uF -> 2.2uF; device LinnesLab-Passives:CAPACITOR0603 -> LinnesLab-Passives:CAPACITOR0402
- C2: value 1u -> 47p
- C20: value 4.7u -> 2.2uF; device LinnesLab-Passives:CAPACITOR0603 -> LinnesLab-Passives:CAPACITOR0402
- C21: value 4.7u -> 1u
- C5: value 1u -> (none)
- C6: value 1u -> 100n
- C7: value 1u -> 4.7u
- C8: value (none) -> 1u
- J1: device LinnesLab-Connectors:CONN_07 -> LinnesLab-Connectors:CONN_07-1.27MM
- LED3: value RED -> YELLOW
- R1, R2: value 0 -> 10k
- R11: value (none) -> 1k
- R14, R15: value 100k -> 0
- R17: value 27 -> 10k
- R18: value 27 -> 390k
- R3, R4: value 1k -> 27
- R5: value 10k -> 100k
- R6: value 10k -> (none)
- R7: value 390k -> 100k
- R8, R9: value 10k -> 1k
- SW1, SW2: value SWITCH.MOM -> (none); device LinnesLab-Switches:SWITCH.MOM -> LinnesLab-Switches:SPST-PTS830GG140-COPY.1-3
- SW3, SW4: value (none) -> SWITCH.MOM; device LinnesLab-Switches:SPST-PTS830GG140-COPY.1-3 -> LinnesLab-Switches:SWITCH.MOM
- U2: value NRF52832_MODULE_MDBT42 -> FT231XS; device LinnesLab-Microcontrollers:NRF52832_MODULE_MDBT42 -> LinnesLab-DigitalIC:FT231XS
- U3: value (none) -> PCF8523; device LinnesLab-Displays:DISP_OLED_UG-2864HSWEG01-NO-WRAPAROUND -> LinnesLab-Clocks:PCF8523; DIGIKEY (none) -> 568-5306-1-ND; I2C_ADDRESS (none) -> 0x68h; MFN (none) -> PCF8523T/1,118; MFN_MANUFACTURER (none) -> NXP USA Inc.
- U4: value PCF8523 -> (none); device LinnesLab-Clocks:PCF8523 -> LinnesLab-Displays:DISP_OLED_UG-2864HSWEG01-NO-WRAPAROUND; DIGIKEY 568-5306-1-ND -> (none); I2C_ADDRESS 0x68h -> (none); MFN PCF8523T/1,118 -> (none); MFN_MANUFACTURER NXP USA Inc. -> (none)
- XTAL2: value 32.768kHz -> 32.7680kHz; FREQ (none) -> 32.7680KHZ
- renumbered C23 to C3, CHRG2 to CHRG1, CORTEX1 to DEBUG1, D5 to D2, JP2 to JP1, L2 to L1, LDO2 to LDO1, LED5 to LED1, R20 to R10, SD2 to SD1, USB2 to USB1
Connections:
- net !CTS: now also U2.!CTS; no longer U5.!CTS
- net 3.3V: now also C12.1, C20.2, C21.1, C4.2, C6.2, D3.C, J1.4, LED3.A, R1.2, R16.2, R2.2, R7.2, U1.VDD, U2.!RESET, U2.VCCIO, U4.VBAT; no longer C12.2, C17.2, C2.1, C22.2, C6.1, D1.C, LED6.A, R15.2, R5.2, R8.2, R9.2, U2.VDD, U3.VBAT, U5.!RESET, U5.VCCIO
- net A4/BATT: now also R12.1, R13.2, U1.P0.28/AIN4; no longer R13.1, R14.2, U2.P0.28/AIN4
- net A6/TIA: now also J1.6, U1.P0.30/AIN6; no longer U2.P0.30/AIN6
- net A7/PPG: now also J1.7, U1.P0.31/AIN7; no longer U2.P0.31/AIN7
- net D11/SW1: now also SW3.1, SW3.2, U1.P0.11; no longer SW1.1, SW1.2, U2.P0.11
- net D15/SW2: now also SW4.1, SW4.2, U1.P0.15; no longer SW2.1, SW2.2, U2.P0.15
- net D16/CS.OLED: now also U1.P0.16, U4./CS; no longer U2.P0.16, U3./CS
- net D27/CHRG.STATUS: now also R5.1, U1.P0.27; no longer R12.1, U2.P0.27
- net D29/LED.CTRL: now also J1.5, U1.P0.29/AIN5; no longer U2.P0.29/AIN5
- net D3/RESET.OLED: now also U1.P0.03/AIN1, U4./RES; no longer U2.P0.03/AIN1, U3./RES
- net D4/DC.OLED: now also U1.P0.04/AIN2, U4.DC/I2C_SA0; no longer U2.P0.04/AIN2, U3.DC/I2C_SA0
- net D5/CD1: now also U1.P0.05/AIN3; no longer U2.P0.05/AIN3
- net D7/SD.CS: now also U1.P0.07; no longer U2.P0.07
- net DFU: now also SW1.B, U1.P0.20; no longer SW3.B, U2.P0.20
- net DTR: now also U2.!DTR; no longer U5.!DTR
- net FRST: now also U1.P0.22; no longer U2.P0.22
- net FT3V3: now also U2.3V3OUT; no longer U5.3V3OUT
- net GND: now also C1.2, C12.2, C13.2, C15.1, C2.1, C20.1, C21.2, C4.1, C6.1, C7.1, J1.3, LED2.C, R13.1, R17.1, R18.2, R7.1, SW1.A, SW2.B, SW3.3, SW3.4, SW4.3, SW4.4, U1.GND@1, U1.GND@2, U1.GND@3, U1.GND@4, U2.GND@16, U2.GND@6, U4.BS0, U4.BS2, U4.NC(GND)@1, U4.NC(GND)@2, U4.VLSS; no longer C12.1, C16.1, C18.1, C2.2, C20.2, C21.1, C22.1, C24.1, C6.2, C7.2, LED3.C, R11.1, R14.1, R15.1, R7.2, SW1.3, SW1.4, SW2.3, SW2.4, SW3.A, SW4.B, U2.GND@1, U2.GND@2, U2.GND@3, U2.GND@4, U3.BS0, U3.BS2, U3.NC(GND)@1, U3.NC(GND)@2, U3.VLSS, U5.GND@16, U5.GND@6
- net LED1: now also R9.2, U1.P0.17; no longer R3.2, U2.P0.17
- net LED2: now also R11.2, U1.P0.19; no longer R4.2, U2.P0.19
- net MISO: now also U1.P0.14; no longer U2.P0.14
- net MOSI: now also U1.P0.13, U4.D1/SPI_SDIN/I2C_SDA; no longer U2.P0.13, U3.D1/SPI_SDIN/I2C_SDA
- net N$1: now also R17.2, U4.BS1; no longer R6.2, U3.BS1
- net N$10: now also R11.1; no longer R4.1
- net N$11: now also U1.DCC; no longer U2.DCC
- net N$12: now also C1.1, U1.DEC4; no longer C7.1, U2.DEC4
- net N$13: now also C15.2, U4.VCC; no longer C16.2, U3.VCC
- net N$15: now also C17.2, U4.VCOMH; no longer C18.2, U3.VCOMH
- net N$17: now also R6.2; no longer R11.2
- net N$2: now also R18.1, U4.IREF; no longer R7.1, U3.IREF
- net N$25: now also U3.OSCO, XTAL2.1; no longer U4.OSCO, XTAL3.1
- net N$26: now also U3.OSCI, XTAL2.2; no longer U4.OSCI, XTAL3.2
- net N$29: now also R3.2, U2.USBDM; no longer R17.2, U5.USBDM
- net N$3: now also C18.2, U4.C2P; no longer C13.2, U3.C2P
- net N$30: now also R4.2, U2.USBDP; no longer R18.2, U5.USBDP
- net N$31: now also R8.2; no longer R19.2
- net N$32: now also LED3.C; no longer LED6.C
- net N$4: now also C5.2, U1.P0.00/XL1, XTAL1.1; no longer C8.2, U2.P0.00/XL1, XTAL2.1
- net N$5: now also C18.1, U4.C2N; no longer C13.1, U3.C2N
- net N$6: now also U1.P0.01/XL2, XTAL1.2; no longer U2.P0.01/XL2, XTAL2.2
- net N$7: now also C16.2, U4.C1P; no longer C15.2, U3.C1P
- net N$8: now also C16.1, U4.C1N; no longer C15.1, U3.C1N
- net N$9: now also LED2.A, R9.1; no longer LED3.A, R3.1
- net P0.09/NFC1: now also C10.1, U1.P0.09; no longer C11.1, U2.P0.09
- net P0.10/NFC2: now also C11.1, U1.P0.10; no longer C10.1, U2.P0.10
- net RESET: now also D3.A, R16.1, SW2.A, U1.P0.21/RESET; no longer D1.A, R5.1, SW4.A, U2.P0.21/RESET
- net RXD.FT: now also R14.1, U2.RXD; no longer R2.1, U5.RXD
- net RXD.NRF: now also R15.2, U1.P0.08; no longer R1.2, U2.P0.08
- net RXLED: now also R8.1, U2.CBUS1; no longer R19.1, U5.CBUS1
- net SCK: now also U1.P0.12, U4.D0/SPI_SCLK/I2C_SCK; no longer U2.P0.12, U3.D0/SPI_SCLK/I2C_SCK
- net SCL: now also J1.2, R2.1, U1.P0.26, U3.SCL; no longer R9.1, U2.P0.26, U4.SCL
- net SDA: now also J1.1, R1.1, U1.P0.25, U3.SDA; no longer R8.1, U2.P0.25, U4.SDA
- net SWCLK: now also U1.SWDCLK; no longer U2.SWDCLK
- net SWDIO: now also U1.SWDIO; no longer U2.SWDIO
- net SWO: now also U1.P0.18/SWO; no longer U2.P0.18/SWO
- net TXD.FT: now also R15.1, U2.TXD; no longer R1.1, U5.TXD
- net TXD.NRF: now also R14.2, U1.P0.06; no longer R2.2, U2.P0.06
- net TXLED: now also U2.CBUS2; no longer U5.CBUS2
- net USB+: now also R4.1; no longer R18.1
- net USB-: now also C2.2, R3.1; no longer C24.2, R17.1
- net VIN: now also C7.2, C8.2, D1.C, R5.2; no longer C21.2, C5.2, D4.C, R12.2
- net VLIPO: now also C13.1, D1.A, R12.2; no longer C20.1, D4.A, R13.2
- net V_USB: now also U2.VCC; no longer U5.VCC
Other:
- moved on the sheet: C10, C11, C12, C13, C15, C16, C17, C18, C2, C20, C21, C5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

Commit message: Take 4 Complete
Parts:
- removed C10, C11: 300p, LinnesLab-Passives:CAPACITOR0603
- removed R7: 100k, LinnesLab-Passives:RESISTOR0603
Connections:
- net 3.3V: no longer R7.2
- net GND: no longer C10.2, C11.2, R7.1, SW3.4, SW4.4
- net P0.09/NFC1: no longer C10.1
- net P0.10/NFC2: no longer C11.1
Changed lines of the file:
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@@
 <part name="GND15" library="LinnesLab-Symbols" deviceset="GND" device=""/>
 <part name="GND16" library="LinnesLab-Symbols" deviceset="GND" device=""/>
-<part name="GND17" library="LinnesLab-Symbols" deviceset="GND" device=""/>
-<part name="GND18" library="LinnesLab-Symbols" deviceset="GND" device=""/>
 <part name="GND19" library="LinnesLab-Symbols" deviceset="GND" device=""/>
 <part name="GND20" library="LinnesLab-Symbols" deviceset="GND" device=""/>
@@
 <part name="C5" library="LinnesLab-Passives" deviceset="CAPACITOR" device="0603" package3d_urn="urn:adsk.eagle:package:15661989/2"/>
 <part name="C9" library="LinnesLab-Passives" deviceset="CAPACITOR" device="0603" package3d_urn="urn:adsk.eagle:package:15661989/2"/>
-<part name="C11" library="LinnesLab-Passives" deviceset="CAPACITOR" device="0603" package3d_urn="urn:adsk.eagle:package:15661989/2" value="300p"/>
-<part name="C10" library="LinnesLab-Passives" deviceset="CAPACITOR" device="0603" package3d_urn="urn:adsk.eagle:package:15661989/2" value="300p"/>
 <part name="C4" library="LinnesLab-Passives" deviceset="CAPACITOR" device="0805" package3d_urn="urn:adsk.eagle:package:15662010/2" value="10u"/>
 <part name="L1" library="LinnesLab-Passives" deviceset="INDUCTOR" device="0603" override_package3d_urn="urn:adsk.eagle:package:18592195/2" override_package_urn="urn:adsk.eagle:footprint:18592196/1" value="10u"/>
@@
 <part name="SUPPLY16" library="LinnesLab-Symbols" deviceset="VLIPO" device=""/>
 <part name="GND43" library="LinnesLab-Symbols" deviceset="GND" device=""/>
-<part name="R7" library="LinnesLab-Passives" deviceset="RESISTOR" device="0603" package3d_urn="urn:adsk.eagle:package:15661944/2" value="100k"/>
-<part name="GND44" library="LinnesLab-Symbols" deviceset="GND" device=""/>
 <part name="SUPPLY17" library="LinnesLab-Symbols" deviceset="VIN" device=""/>
 <part name="SW3" library="LinnesLab-Switches" deviceset="SWITCH.MOM" device=""/>
@@
 <attribute name="VALUE" x="121.92" y="42.926" size="1.778" layer="96" align="top-center"/>
 </instance>
-<instance part="GND17" gate="G$1" x="124.46" y="12.7" smashed="yes">
-<attribute name="VALUE" x="124.46" y="12.446" size="1.778" layer="96" align="top-center"/>
-</instance>
-<instance part="GND18" gate="G$1" x="111.76" y="12.7" smashed="yes">
-<attribute name="VALUE" x="111.76" y="12.446" size="1.778" layer="96" align="top-center"/>
-</instance>
 <instance part="GND19" gate="G$1" x="101.6" y="12.7" smashed="yes">
 <attribute name="VALUE" x="101.6" y="12.446" size="1.778" layer="96" align="top-center"/>
@@
 <attribute name="VALUE" x="103.124" y="18.161" size="1.778" layer="96"/>
 </instance>
-<instance part="C11" gate="G$1" x="124.46" y="20.32" smashed="yes">
-<attribute name="NAME" x="125.984" y="23.241" size="1.778" layer="95"/>
-<attribute name="VALUE" x="125.984" y="18.161" size="1.778" layer="96"/>
-</instance>
-<instance part="C10" gate="G$1" x="111.76" y="20.32" smashed="yes">
-<attribute name="NAME" x="113.284" y="23.241" size="1.778" layer="95"/>
-<attribute name="VALUE" x="113.284" y="18.161" size="1.778" layer="96"/>
-</instance>
 <instance part="C4" gate="G$1" x="81.28" y="55.88" smashed="yes" rot="R180">
 <attribute name="NAME" x="79.756" y="52.959" size="1.778" layer="95" rot="R180"/>
@@
 <instance part="GND43" gate="G$1" x="129.54" y="-134.62" smashed="yes">
 <attribute name="VALUE" x="129.54" y="-134.874" size="1.778" layer="96" align="top-center"/>
-</instance>
-<instance part="R7" gate="G$1" x="142.24" y="-99.06" smashed="yes" rot="R90">
-<attribute name="NAME" x="140.7414" y="-102.87" size="1.778" layer="95" rot="R90"/>
-<attribute name="VALUE" x="145.542" y="-102.87" size="1.778" layer="96" rot="R90"/>
-</instance>
-<instance part="GND44" gate="G$1" x="142.24" y="-109.22" smashed="yes">
-<attribute name="VALUE" x="142.24" y="-109.474" size="1.778" layer="96" align="top-center"/>
 </instance>
 <instance part="SUPPLY17" gate="G$1" x="83.82" y="-88.9" smashed="yes">
@@
 <pinref part="GND20" gate="G$1" pin="GND"/>
 <pinref part="C5" gate="G$1" pin="1"/>
-</segment>
-<segment>
-<pinref part="C10" gate="G$1" pin="2"/>
-<pinref part="GND18" gate="G$1" pin="GND"/>
-<wire x1="111.76" y1="15.24" x2="111.76" y2="17.78" width="0.1524" layer="91"/>
-</segment>
-<segment>
-<pinref part="C11" gate="G$1" pin="2"/>
-<pinref part="GND17" gate="G$1" pin="GND"/>
-<wire x1="124.46" y1="15.24" x2="124.46" y2="17.78" width="0.1524" layer="91"/>
 </segment>
 <segment>
@@
 </segment>
 <segment>
-<pinref part="R7" gate="G$1" pin="1"/>
-<pinref part="GND44" gate="G$1" pin="GND"/>
-<wire x1="142.24" y1="-106.68" x2="142.24" y2="-104.14" width="0.1524" layer="91"/>
-</segment>
-<segment>
 <pinref part="SW3" gate="G$1" pin="3"/>
 <wire x1="378.46" y1="-73.66" x2="386.08" y2="-73.66" width="0.1524" layer="91"/>
-<wire x1="386.08" y1="-73.66" x2="386.08" y2="-76.2" width="0.1524" layer="91"/>
-<pinref part="SW3" gate="G$1" pin="4"/>
-<wire x1="386.08" y1="-91.44" x2="386.08" y2="-76.2" width="0.1524" layer="91"/>
-<wire x1="386.08" y1="-76.2" x2="378.46" y2="-76.2" width="0.1524" layer="91"/>
+<wire x1="386.08" y1="-91.44" x2="386.08" y2="-73.66" width="0.1524" layer="91"/>
 <pinref part="GND1" gate="G$1" pin="GND"/>
 </segment>
@@
 <pinref part="SW4" gate="G$1" pin="3"/>
 <wire x1="421.64" y1="-58.42" x2="429.26" y2="-58.42" width="0.1524" layer="91"/>
-<wire x1="429.26" y1="-58.42" x2="429.26" y2="-60.96" width="0.1524" layer="91"/>
-<pinref part="SW4" gate="G$1" pin="4"/>
-<wire x1="429.26" y1="-76.2" x2="429.26" y2="-60.96" width="0.1524" layer="91"/>
-<wire x1="429.26" y1="-60.96" x2="421.64" y2="-60.96" width="0.1524" layer="91"/>
+<wire x1="429.26" y1="-76.2" x2="429.26" y2="-58.42" width="0.1524" layer="91"/>
 <pinref part="GND3" gate="G$1" pin="GND"/>
 </segment>
@@
 <wire x1="132.08" y1="-88.9" x2="132.08" y2="-91.44" width="0.1524" layer="91"/>
 <junction x="132.08" y="-91.44"/>
-<wire x1="132.08" y1="-91.44" x2="142.24" y2="-91.44" width="0.1524" layer="91"/>
-<pinref part="R7" gate="G$1" pin="2"/>
-<wire x1="142.24" y1="-91.44" x2="142.24" y2="-93.98" width="0.1524" layer="91"/>
 </segment>
 <segment>
@@
 <segment>
 <wire x1="116.84" y1="48.26" x2="116.84" y2="27.94" width="0.1524" layer="91"/>
-<wire x1="111.76" y1="27.94" x2="116.84" y2="27.94" width="0.1524" layer="91"/>
-<wire x1="111.76" y1="27.94" x2="111.76" y2="25.4" width="0.1524" layer="91"/>
-<pinref part="C10" gate="G$1" pin="1"/>
 <pinref part="U1" gate="G$1" pin="P0.09"/>
 <label x="116.84" y="30.48" size="1.27" layer="95" rot="R180" xref="yes"/>
@@
 <segment>
 <wire x1="119.38" y1="48.26" x2="119.38" y2="27.94" width="0.1524" layer="91"/>
-<wire x1="119.38" y1="27.94" x2="124.46" y2="27.94" width="0.1524" layer="91"/>
-<wire x1="124.46" y1="27.94" x2="124.46" y2="25.4" width="0.1524" layer="91"/>
-<pinref part="C11" gate="G$1" pin="1"/>
 <pinref part="U1" gate="G$1" pin="P0.10"/>
 <label x="119.38" y="30.48" size="1.27" layer="95" xref="yes"/>

Commit message: Take 06
Parts:
- removed C12, C21, C8: 1u, LinnesLab-Passives:CAPACITOR0603
- removed C13, C7: 4.7u, LinnesLab-Passives:CAPACITOR0603
- removed CHRG1: MCP73831, LinnesLab-Power:MCP73831
- removed LDO1: MIC5504, LinnesLab-Power:MIC5504
- removed R5: 100k, LinnesLab-Passives:RESISTOR0603
- removed R6: (no value), LinnesLab-Passives:RESISTOR0603
- removed SD1: (no value), LinnesLab-Connectors:MICROSD
- removed U3: PCF8523, LinnesLab-Clocks:PCF8523
- removed XTAL2: 32.7680kHz, LinnesLab-Clocks:CRYSTALECS-.327-12.5-12-C-TR
Connections:
- removed net CD2: SD1.CARD_DETECT1
- removed net N$17: CHRG1.PROG, R6.2
- removed net N$25: U3.OSCO, XTAL2.1
- removed net N$26: U3.OSCI, XTAL2.2
- net 3.3V: no longer C12.1, C21.1, LDO1.OUT, SD1.VDD, U3.VDD
- net D27/CHRG.STATUS: no longer CHRG1.STAT, R5.1
- net D5/CD1: no longer SD1.CARD_DETECT
- net D7/SD.CS: no longer SD1.CS
- net GND: no longer C12.2, C13.2, C21.2, C7.1, C8.1, CHRG1.VSS, LDO1.GND, R6.1, SD1.GND, SD1.GND1, SD1.VSS, U3.VSS
- net MISO: no longer SD1.DATA_OUT
- net MOSI: no longer SD1.DATA_IN
- net SCK: no longer SD1.SCLK
- net SCL: no longer U3.SCL
- net SDA: no longer U3.SDA
- net VIN: no longer C7.2, C8.2, CHRG1.VIN, LDO1.EN, LDO1.IN, R5.2
- net VLIPO: no longer C13.1, CHRG1.VBAT
Other:
- note removed: "Back-up battery if desired"
- note removed: "Connect MISO, MOSI, and SCK to appropriate pins on microcontroller. Those are SPI pins and are generally prespecified. You have more flexibility with the SD.CS pin."
- note removed: "I2C Address = 0x68h"

Commit message: Take 7
Parts:
- C17: device LinnesLab-Passives:CAPACITOR0402 -> LinnesLab-Passives:CAPACITOR0603
Connections:
- removed net A4/BATT: R12.1, R13.2, U1.P0.28/AIN4
- removed net A6/TIA: J1.6, U1.P0.30/AIN6
- removed net A7/PPG: J1.7, U1.P0.31/AIN7
- removed net D29/LED.CTRL: J1.5, U1.P0.29/AIN5
- new net A4/PPG: J1.7, U1.P0.28/AIN4
- new net A5/TIA: J1.6, U1.P0.29/AIN5
- new net A7/BATT: R12.1, R13.2, U1.P0.31/AIN7
- new net D30/LED.CTRL: J1.5, U1.P0.30/AIN6
Changed lines of the file:
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@@
 <part name="C15" library="LinnesLab-Passives" deviceset="CAPACITOR" device="0603" package3d_urn="urn:adsk.eagle:package:15661989/2" value="10uF"/>
 <part name="C20" library="LinnesLab-Passives" deviceset="CAPACITOR" device="0402" package3d_urn="urn:adsk.eagle:package:15402268/2" value="2.2uF"/>
-<part name="C17" library="LinnesLab-Passives" deviceset="CAPACITOR" device="0402" package3d_urn="urn:adsk.eagle:package:15402268/2" value="2.2uF"/>
+<part name="C17" library="LinnesLab-Passives" deviceset="CAPACITOR" device="0603" package3d_urn="urn:adsk.eagle:package:15661989/2" value="2.2uF"/>
 <part name="C19" library="LinnesLab-Passives" deviceset="CAPACITOR" device="0402" package3d_urn="urn:adsk.eagle:package:15402268/2" value="2.2uF"/>
 <part name="U4" library="LinnesLab-Displays" deviceset="DISP_OLED_UG-2864HSWEG01" device="-NO-WRAPAROUND"/>
@@
 </segment>
 </net>
-<net name="A4/BATT" class="0">
-<segment>
-<pinref part="U1" gate="G$1" pin="P0.28/AIN4"/>
-<wire x1="83.82" y1="78.74" x2="81.28" y2="78.74" width="0.1524" layer="91"/>
-<label x="81.28" y="78.74" size="1.27" layer="95" rot="R180" xref="yes"/>
-</segment>
-<segment>
-<pinref part="R12" gate="G$1" pin="1"/>
-<pinref part="R13" gate="G$1" pin="2"/>
-<wire x1="160.02" y1="-114.3" x2="160.02" y2="-106.68" width="0.1524" layer="91"/>
-<label x="160.02" y="-111.76" size="1.27" layer="95" xref="yes"/>
-</segment>
-</net>
-<net name="D29/LED.CTRL" class="0">
-<segment>
-<pinref part="U1" gate="G$1" pin="P0.29/AIN5"/>
-<wire x1="83.82" y1="76.2" x2="81.28" y2="76.2" width="0.1524" layer="91"/>
-<label x="81.28" y="76.2" size="1.27" layer="95" rot="R180" xref="yes"/>
-</segment>
-<segment>
-<pinref part="J1" gate="G$1" pin="5"/>
-<wire x1="-30.48" y1="213.36" x2="-22.86" y2="213.36" width="0.1524" layer="91"/>
-<label x="-22.86" y="213.36" size="1.778" layer="95" xref="yes"/>
-</segment>
-</net>
-<net name="A6/TIA" class="0">
-<segment>
-<pinref part="U1" gate="G$1" pin="P0.30/AIN6"/>
-<wire x1="83.82" y1="73.66" x2="81.28" y2="73.66" width="0.1524" layer="91"/>
-<label x="81.28" y="73.66" size="1.27" layer="95" rot="R180" xref="yes"/>
-</segment>
-<segment>
-<pinref part="J1" gate="G$1" pin="6"/>
-<wire x1="-30.48" y1="215.9" x2="-22.86" y2="215.9" width="0.1524" layer="91"/>
-<label x="-22.86" y="215.9" size="1.778" layer="95" xref="yes"/>
-</segment>
-</net>
 <net name="N$29" class="0">
 <segment>
@@
 </segment>
 </net>
-<net name="A7/PPG" class="0">
+<net name="A4/PPG" class="0">
+<segment>
+<pinref part="U1" gate="G$1" pin="P0.28/AIN4"/>
+<wire x1="83.82" y1="78.74" x2="81.28" y2="78.74" width="0.1524" layer="91"/>
+<label x="81.28" y="78.74" size="1.27" layer="95" rot="R180" xref="yes"/>
+</segment>
+<segment>
+<pinref part="J1" gate="G$1" pin="7"/>
+<wire x1="-30.48" y1="218.44" x2="-22.86" y2="218.44" width="0.1524" layer="91"/>
+<label x="-22.86" y="218.44" size="1.778" layer="95" xref="yes"/>
+</segment>
+</net>
+<net name="A7/BATT" class="0">
 <segment>
 <pinref part="U1" gate="G$1" pin="P0.31/AIN7"/>
@@
 </segment>
 <segment>
-<pinref part="J1" gate="G$1" pin="7"/>
-<wire x1="-30.48" y1="218.44" x2="-22.86" y2="218.44" width="0.1524" layer="91"/>
-<label x="-22.86" y="218.44" size="1.778" layer="95" xref="yes"/>
-</segment>
-</net>
+<pinref part="R12" gate="G$1" pin="1"/>
+<pinref part="R13" gate="G$1" pin="2"/>
+<wire x1="160.02" y1="-114.3" x2="160.02" y2="-106.68" width="0.1524" layer="91"/>
+<label x="160.02" y="-111.76" size="1.27" layer="95" xref="yes"/>
+</segment>
+</net>
+<net name="D30/LED.CTRL" class="0">
+<segment>
+<pinref part="U1" gate="G$1" pin="P0.30/AIN6"/>
+<wire x1="83.82" y1="73.66" x2="81.28" y2="73.66" width="0.1524" layer="91"/>
+<label x="81.28" y="73.66" size="1.27" layer="95" rot="R180" xref="yes"/>
+</segment>
+<segment>
+<pinref part="J1" gate="G$1" pin="5"/>
+<wire x1="-30.48" y1="213.36" x2="-22.86" y2="213.36" width="0.1524" layer="91"/>
+<label x="-22.86" y="213.36" size="1.778" layer="95" xref="yes"/>
+</segment>
+</net>
+<net name="A5/TIA" class="0">
+<segment>
+<pinref part="U1" gate="G$1" pin="P0.29/AIN5"/>
+<wire x1="83.82" y1="76.2" x2="81.28" y2="76.2" width="0.1524" layer="91"/>
+<label x="81.28" y="76.2" size="1.27" layer="95" rot="R180" xref="yes"/>
+</segment>
+<segment>
+<pinref part="J1" gate="G$1" pin="6"/>
+<wire x1="-30.48" y1="215.9" x2="-22.86" y2="215.9" width="0.1524" layer="91"/>
+<label x="-22.86" y="215.9" size="1.778" layer="95" xref="yes"/>
+</segment>
+</net>
