File: Hardware/Basic/Top/LowKey-BASIC-TOP.sch (EAGLE design)
At the start: 51 parts, among them SW3 SWITCH.MOM, SW4 SWITCH.MOM, SW5 SWITCH.MOM, U1 NRF52832_MODULE_MDBT42, U2 FT231XS

Commit message: Finished routing top board
Parts:
- removed C19, C20: 2.2uF, LinnesLab-Passives:CAPACITOR0402
- removed SW5: SWITCH.MOM, LinnesLab-Switches:SWITCH.MOM
- added C10: 1u, LinnesLab-Passives:CAPACITOR0603
- added C11, C8: 4.7u, LinnesLab-Passives:CAPACITOR0603
- added C12: 100n, LinnesLab-Passives:CAPACITOR0603
- added C13: 10uF, LinnesLab-Passives:CAPACITOR0603
- added C7: (no value), LinnesLab-Passives:CAPACITOR0603
- added CHRG1: MCP73831, LinnesLab-Power:MCP73831
- added LDO1: MIC5504, LinnesLab-Power:MIC5504
- added R5: 100k, LinnesLab-Passives:RESISTOR0603
- added R6, R7: 1k, LinnesLab-Passives:RESISTOR0603
- C14: value 100n -> 2.2uF; device LinnesLab-Passives:CAPACITOR0603 -> LinnesLab-Passives:CAPACITOR0402
- C15: value 10uF -> 2.2uF
- C17: device LinnesLab-Passives:CAPACITOR0603 -> LinnesLab-Passives:CAPACITOR0402
- C9: value (none) -> 1u
- R10: value 1k -> 100k
- R8: value 1k -> (none)
- renumbered U4 to U3
Connections:
- removed net D27/CHRG.STATUS: U1.P0.27
- removed net SW3: SW5.1, SW5.2
- new net D27/CHRG.STAT: CHRG1.STAT, R5.1, U1.P0.27
- new net N$17: CHRG1.PROG, R8.2
- net 3.3V: now also C10.1, C17.2, C18.2, LDO1.OUT, R10.2; no longer C19.2, C20.2
- net DTR: now also C12.1; no longer C14.1
- net GND: now also C10.2, C11.2, C13.1, C18.1, C7.2, C8.1, C9.1, CHRG1.VSS, LDO1.GND, R10.1, R8.1; no longer C19.1, C20.1, C9.2, SW5.3, SW5.4
- net LED1: now also R7.2; no longer R9.2
- net N$13: now also C13.2; no longer C15.2
- net N$15: now also C15.2; no longer C17.2
- net N$3: now also C16.2; no longer C18.2
- net N$31: now also R6.2; no longer R8.2
- net N$32: now also R9.2; no longer R10.2
- net N$5: now also C16.1; no longer C18.1
- net N$6: now also C7.1; no longer C9.1
- net N$7: now also C14.2; no longer C16.2
- net N$8: now also C14.1; no longer C16.1
- net N$9: now also R7.1; no longer R9.1
- net RESET: now also C12.2; no longer C14.2
- net RXLED: now also R6.1; no longer R8.1
- net TXLED: now also R9.1; no longer R10.1
- net VIN: now also C8.2, C9.2, CHRG1.VIN, LDO1.EN, LDO1.IN, R5.2
- net VLIPO: now also C11.1, CHRG1.VBAT
Other:
- moved on the sheet: C14, C15, C16, C17, C18, C9, R10, R12, R13, R8, R9
